Commit message: Add dual JAKA A12 Gazebo bringup and dual trajectory backend

File: src/jaka_ros2/src/jaka_a12_moveit_config/config/jaka_a12_prefixed.urdf.xacro (robot description, xacro)
@@ -2,6 +2,19 @@
 <robot xmlns:xacro="http://www.ros.org/wiki/xacro">
   <xacro:property name="jaka_a12_mesh_path" value="package://jaka_description/meshes/jaka_a12_meshes"/>
-  <xacro:macro name="jaka_a12_prefixed" params="prefix parent:=world base_xyz:='0 0 0' base_rpy:='0 0 0'">
+  <xacro:macro name="jaka_a12_prefixed" params="prefix parent:=world base_xyz:='0 0 0' base_rpy:='0 0 0' include_inertial:=false">
     <link name="${prefix}base_link">
+      <xacro:if value="${include_inertial}">
+        <inertial>
+          <origin xyz="0.00016274 2.3475E-05 0.017516" rpy="0 0 0"/>
+          <mass value="0.84938"/>
+          <inertia
+            ixx="0.0015415"
+            ixy="5.5705E-08"
+            ixz="-1.6043E-07"
+            iyy="0.0018861"
+            iyz="2.6186E-07"
+            izz="0.0032224"/>
+        </inertial>
+      </xacro:if>
       <visual>
         <origin xyz="0 0 0" rpy="0 0 0"/>
@@ -26,4 +39,17 @@
     </joint>
     <link name="${prefix}J1">
+      <xacro:if value="${include_inertial}">
+        <inertial>
+          <origin xyz="6.0416E-08 -0.0029272 -0.004247" rpy="0 0 0"/>
+          <mass value="3.7579"/>
+          <inertia
+            ixx="0.01765"
+            ixy="-2.5806E-07"
+            ixz="-1.3081E-07"
+            iyy="0.017355"
+            iyz="3.4234E-05"
+            izz="0.011502"/>
+        </inertial>
+      </xacro:if>
       <visual>
         <origin xyz="0 0 0" rpy="0 0 0"/>
@@ -50,4 +76,17 @@
     </joint>
     <link name="${prefix}J2">
+      <xacro:if value="${include_inertial}">
+        <inertial>
+          <origin xyz="0.32342 7.7419E-08 0.1801" rpy="0 0 0"/>
+          <mass value="13.37"/>
+          <inertia
+            ixx="0.038258"
+            ixy="3.482E-08"
+            ixz="-0.0030725"
+            iyy="1.0882"
+            iyz="5.5423E-08"
+            izz="1.0803"/>
+        </inertial>
+      </xacro:if>
       <visual>
         <origin xyz="0 0 0" rpy="0 0 0"/>
@@ -74,4 +113,17 @@
     </joint>
     <link name="${prefix}J3">
+      <xacro:if value="${include_inertial}">
+        <inertial>
+          <origin xyz="-4.2655E-07 -0.0024273 0.002914" rpy="0 0 0"/>
+          <mass value="1.9435"/>
+          <inertia
+            ixx="0.0057394"
+            ixy="3.386E-10"
+            ixz="7.7883E-08"
+            iyy="0.0038913"
+            iyz="3.3725E-06"
+            izz="0.0056521"/>
+        </inertial>
+      </xacro:if>
       <visual>
         <origin xyz="0 0 0" rpy="0 0 0"/>
@@ -98,4 +150,17 @@
     </joint>
     <link name="${prefix}J4">
+      <xacro:if value="${include_inertial}">
+        <inertial>
+          <origin xyz="3.1406E-08 -0.00097336 -0.21333" rpy="0 0 0"/>
+          <mass value="3.903"/>
+          <inertia
+            ixx="0.10135"
+            ixy="4.9565E-08"
+            ixz="-9.9161E-09"
+            iyy="0.10077"
+            iyz="0.00080984"
+            izz="0.0051085"/>
+        </inertial>
+      </xacro:if>
       <visual>
         <origin xyz="0 0 0" rpy="0 0 0"/>
@@ -122,4 +187,17 @@
     </joint>
     <link name="${prefix}J5">
+      <xacro:if value="${include_inertial}">
+        <inertial>
+          <origin xyz="1.1338E-07 0.0049095 -0.0024985" rpy="0 0 0"/>
+          <mass value="1.0253"/>
+          <inertia
+            ixx="0.0022543"
+            ixy="1.8791E-09"
+            ixz="1.7943E-08"
+            iyy="0.0011832"
+            iyz="-1.3434E-05"
+            izz="0.0022184"/>
+        </inertial>
+      </xacro:if>
       <visual>
         <origin xyz="0 0 0" rpy="0 0 0"/>
@@ -146,4 +224,17 @@
     </joint>
     <link name="${prefix}J6">
+      <xacro:if value="${include_inertial}">
+        <inertial>
+          <origin xyz="-6.1189E-05 -5.6233E-05 -0.020571" rpy="0 0 0"/>
+          <mass value="0.2135"/>
+          <inertia
+            ixx="0.00012541"
+            ixy="4.199E-07"
+            ixz="-2.6224E-08"
+            iyy="0.00012595"
+            iyz="-1.6646E-07"
+            izz="0.00021163"/>
+        </inertial>
+      </xacro:if>
       <visual>
         <origin xyz="0 0 0" rpy="0 0 0"/>
