Commit message: feat: complete integrated dual-arm digital twin through phase 5

File: dual_arm_app/web/assets/dual_jaka_a12_web.urdf (robot description, URDF)
Before this commit: robot dual_jaka_a12, 15 links, 14 joints
Joints:
- joint left_fixed: origin xyz=0.0 0.075 1.2 rpy=1.570796326795 0.0 3.14159265359 -> xyz=-0.759623984260727 0.110586943833874 0.136510144598804 rpy=1.57443900609587 0.00157870658316782 3.14115595321641
- joint right_fixed: origin xyz=0.0 -0.075 1.2 rpy=-1.570796326795 0.0 3.14159265359 -> xyz=-0.762701204626243 -0.0717851558956737 0.134522498785659 rpy=-1.57111248148528 0.00733114096125062 -3.14115515910762

File: src/jaka_ros2/src/jaka_a12_moveit_config/config/dual_jaka_a12.urdf.xacro (robot description, xacro)
@@ -2,14 +2,20 @@
 <robot xmlns:xacro="http://www.ros.org/wiki/xacro" name="dual_jaka_a12">
   <xacro:include filename="$(find jaka_a12_moveit_config)/config/jaka_a12_prefixed.urdf.xacro"/>
+  <!-- Required canonical-calibration inputs. Empty values intentionally fail
+       Xacro processing rather than falling back to duplicated model constants. -->
+  <xacro:arg name="left_base_xyz" default=""/>
+  <xacro:arg name="left_base_rpy" default=""/>
+  <xacro:arg name="right_base_xyz" default=""/>
+  <xacro:arg name="right_base_rpy" default=""/>
   <link name="world"/>
   <xacro:jaka_a12_prefixed
     prefix="left_"
     parent="world"
-    base_xyz="0.0 0.075 1.2"
-    base_rpy="1.570796326795 0.0 3.14159265359"/>
+    base_xyz="$(arg left_base_xyz)"
+    base_rpy="$(arg left_base_rpy)"/>
   <xacro:jaka_a12_prefixed
     prefix="right_"
     parent="world"
-    base_xyz="0.0 -0.075 1.2"
-    base_rpy="-1.570796326795 0.0 3.14159265359"/>
+    base_xyz="$(arg right_base_xyz)"
+    base_rpy="$(arg right_base_rpy)"/>
 </robot>
